File: Kicad Files/Board/Board.kicad_pcb (KiCad board)
At the start: 2 copper layers, 134 parts, among them U1 RP2040-ZERO

Commit message: Switch Update
Parts:
- added D66: D_Small, mechanical_keyboard:D_0402_1005Metric, B.Cu at (356.9, 101.7)
- added MX66: Delete, mechanical_keyboard:SW_Cherry_MX_1.00u_PCB, F.Cu at (349.9, 96.7)
- D1, D10, D11, D12, D13, D14, D15, D16, D17, D18, D19, D2, D20, D21, D22, D23, D24, D25, D26, D27, D28, D29, D3, D30, D31, D32, D33, D34, D35, D36, D37, D38, D39, D4, D40, D41, D42, D43, D44, D45, D46, D47, D48, D49, D5, D50, D51, D52, D53, D54, D55, D56, D57, D58, D59, D6, D60, D61, D62, D63, D64, D65, D7, D8, D9: moved to B.Cu
- MX1, MX10, MX11, MX12, MX13, MX14, MX15, MX16, MX17, MX18, MX19, MX2, MX20, MX21, MX22, MX23, MX24, MX25, MX26, MX27, MX28, MX29, MX3, MX30, MX31, MX32, MX33, MX34, MX35, MX36, MX37, MX38, MX39, MX4, MX40, MX41, MX42, MX43, MX44, MX45, MX46, MX47, MX48, MX49, MX5, MX50, MX51, MX52, MX53, MX54, MX55, MX56, MX57, MX58, MX6, MX62, MX63, MX64, MX65, MX7, MX8, MX9: footprint mechanical_keyboard:SW_MX_1u -> mechanical_keyboard:SW_Cherry_MX_1.00u_PCB
- MX59: value Mode -> RAlt; footprint mechanical_keyboard:SW_MX_1u -> mechanical_keyboard:SW_Cherry_MX_1.00u_PCB
- MX60: value Delete -> Mode; footprint mechanical_keyboard:SW_MX_1u -> mechanical_keyboard:SW_Cherry_MX_1.00u_PCB
- MX61: value Sleep -> LCtrl; footprint mechanical_keyboard:SW_MX_1u -> mechanical_keyboard:SW_Cherry_MX_1.00u_PCB
- moved R8 438.7 mm to (393.2, 83.0)
- moved D72 438.7 mm to (393.8, 78.2)
- moved D73 438.7 mm to (393.8, 80.8)
- moved U1 432.3 mm to (375.1, 86.3)
- moved MX62 91.3 mm to (349.9, 77.6)
- moved D62 85.6 mm to (356.9, 82.7)
- moved MX60 7.18 mm to (268.7, 153.8)
- moved MX59 7.18 mm to (249.7, 153.8)
- moved MX61 7.18 mm to (287.8, 153.8)
- moved MX58 7.14 mm to (180.6, 153.8)
- moved D59 6.87 mm to (256.7, 158.9)
- moved D60 6.87 mm to (275.7, 158.9)
- moved D61 6.87 mm to (294.8, 158.9)
- moved D11 5.68 mm to (256.6, 82.7)
- moved D12 5.68 mm to (275.7, 82.7)
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Connections:
- D62 pad 1: ROW4 -> ROW2
- MX62 pad 1: COL10 -> COL13
- MX63 pad 1: COL11 -> COL10
- MX64 pad 1: COL12 -> COL11
- MX65 pad 1: COL13 -> COL12

Commit message: Silkscreen updated
Parts:
- moved D58 7.15 mm to (187.6, 158.9)

Commit message: Routing Completed
Parts:
- removed D72, D73: LED_Small, mechanical_keyboard:LED_0603_1608Metric
- removed R8: 1K, mechanical_keyboard:R_0402_1005Metric
- moved U1 37.6 mm to (338.1, 80.1)
- moved D65 24.0 mm to (371.0, 158.9)
- moved D54 24.0 mm to (351.9, 139.8)
- moved D63 24.0 mm to (332.9, 158.9)
- moved D64 24.0 mm to (351.9, 158.9)
- moved MX54 24.0 mm to (344.9, 134.8)
- moved MX63 24.0 mm to (325.9, 153.8)
- moved MX64 24.0 mm to (344.9, 153.8)
- moved MX65 24.0 mm to (364.0, 153.8)
- moved D66 14.1 mm to (371.0, 101.6)
- moved D62 14.1 mm to (371.0, 82.7)
- moved MX62 14.1 mm to (364.0, 77.6)
- moved MX66 14.1 mm to (364.0, 96.7)
Connections:
- D62 pad 1: ROW2 -> ROW0
- D66 pad 1: ROW3 -> ROW1
- MX54 pad 1: COL12 -> COL13
- MX58 pad 1: COL3 -> COL5
- MX59 pad 1: COL7 -> COL8
- MX60 pad 1: COL8 -> COL9
- MX61 pad 1: COL9 -> COL10
- MX62 pad 1: COL13 -> COL14
- MX63 pad 1: COL10 -> COL11
- MX64 pad 1: COL11 -> COL13
- MX65 pad 1: COL12 -> COL14
- MX66 pad 1: COL13 -> COL14
- U1 pad 1: unconnected-(U1-GP0-Pad1) -> ROW4
- U1 pad 10: unconnected-(U1-GP9-Pad10) -> COL10
- U1 pad 11: unconnected-(U1-GP10-Pad11) -> COL9
- U1 pad 12: unconnected-(U1-GP11-Pad12) -> COL8
- U1 pad 13: unconnected-(U1-GP12-Pad13) -> COL7
- U1 pad 14: unconnected-(U1-GP13-Pad14) -> COL6
- U1 pad 15: unconnected-(U1-GP14-Pad15) -> COL5
- U1 pad 16: unconnected-(U1-GP15-Pad16) -> COL4
- U1 pad 17: unconnected-(U1-GP26-Pad17) -> COL3
- U1 pad 18: unconnected-(U1-GP27-Pad18) -> COL2
- U1 pad 19: unconnected-(U1-GP28-Pad19) -> COL1
- U1 pad 2: unconnected-(U1-GP1-Pad2) -> ROW3
- U1 pad 20: unconnected-(U1-GP29-Pad20) -> COL0
- U1 pad 3: unconnected-(U1-GP2-Pad3) -> COL14
- U1 pad 4: unconnected-(U1-GP3-Pad4) -> ROW1
- U1 pad 5: unconnected-(U1-GP4-Pad5) -> ROW2
- U1 pad 6: unconnected-(U1-GP5-Pad6) -> ROW0
- U1 pad 7: unconnected-(U1-GP6-Pad7) -> COL13
- U1 pad 8: unconnected-(U1-GP7-Pad8) -> COL12
- U1 pad 9: unconnected-(U1-GP8-Pad9) -> COL11
Routing:
- net ROW4: track 0.00 -> 459.9 mm, vias 0 -> 10
- net ROW3: track 0.00 -> 425.7 mm, vias 0 -> 13
- net ROW1: track 0.00 -> 395.0 mm, vias 0 -> 15
- net COL0: track 0.00 -> 383.8 mm
- net COL1: track 0.00 -> 374.9 mm
- net ROW0: track 0.00 -> 373.9 mm, vias 0 -> 15
- net COL2: track 0.00 -> 365.0 mm
- net ROW2: track 0.00 -> 351.7 mm, vias 0 -> 15
- net COL3: track 0.00 -> 319.8 mm
- net COL5: track 0.00 -> 304.8 mm
- net COL4: track 0.00 -> 301.9 mm
- net COL6: track 0.00 -> 271.1 mm
- net COL8: track 0.00 -> 266.8 mm
- net COL7: track 0.00 -> 253.8 mm
- net COL9: track 0.00 -> 251.9 mm
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Other:
- board outline added: 339.9 x 107.4 mm
